File: pcb/c51keypad/c51keypad.kicad_pcb (KiCad board)
At the start: 2 copper layers, 76.2 x 95.2 mm, 46 parts, among them CN1 PZ254V-11-04P, J1 USB_C_Receptacle_USB2.0_16P, U1 CH9328, U2 STC12C5604AD-35I-DIP20

Commit message: stc15
Parts:
- removed C3: 10uF, Capacitor_SMD:C_0603_1608Metric_Pad1.08x0.95mm_HandSolder
- removed R3: 1k, Resistor_SMD:R_0603_1608Metric_Pad0.98x0.95mm_HandSolder
- removed U2: STC12C5604AD-35I-DIP20, Package_DIP:DIP-20_W7.62mm_Socket_LongPads
- C1, C2, C4, C5, J1, R1, R2, U1: moved to B.Cu
- moved J1 134.7 mm to (38.2, -90.9)
- moved SW13 130.4 mm to (9.61, -28.8)
- moved SW17 112.6 mm to (19.1, -9.78)
- moved U1 110.8 mm to (66.2, -72.0), turned to 90 degrees
- moved SW14 106.9 mm to (28.7, -28.8)
- moved SW9 101.4 mm to (9.61, -47.9)
- moved CN1 97.5 mm to (66.3, -6.57)
- moved C1 90.5 mm to (80.5, -74.6), turned to 180 degrees
- moved C2 90.5 mm to (80.5, -72.1), turned to 180 degrees
- moved C4 90.5 mm to (80.5, -67.1), turned to 180 degrees
- moved C5 90.5 mm to (80.5, -64.6), turned to 180 degrees
- moved R1 90.5 mm to (85.1, -74.4), turned to 180 degrees
- moved R2 90.5 mm to (85.1, -71.4), turned to 180 degrees
- moved SW16 89.2 mm to (47.7, -9.80)
- moved SW5 88.0 mm to (9.61, -66.9)
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Connections:
- J1 pad 13: (no net) -> GND
- SW1 pad 0: (no net) -> unconnected-(SW1-GND-Pad0)
- SW10 pad 0: (no net) -> unconnected-(SW10-GND-Pad0)
- SW11 pad 0: (no net) -> unconnected-(SW11-GND-Pad0)
- SW12 pad 0: (no net) -> unconnected-(SW12-GND-Pad0)
- SW13 pad 0: (no net) -> unconnected-(SW13-GND-Pad0)
- SW14 pad 0: (no net) -> unconnected-(SW14-GND-Pad0)
- SW15 pad 0: (no net) -> unconnected-(SW15-GND-Pad0)
- SW16 pad 0: (no net) -> unconnected-(SW16-GND-Pad0)
- SW17 pad 0: (no net) -> unconnected-(SW17-GND-Pad0)
- SW2 pad 0: (no net) -> unconnected-(SW2-GND-Pad0)
- SW3 pad 0: (no net) -> unconnected-(SW3-GND-Pad0)
- SW4 pad 0: (no net) -> unconnected-(SW4-GND-Pad0)
- SW5 pad 0: (no net) -> unconnected-(SW5-GND-Pad0)
- SW6 pad 0: (no net) -> unconnected-(SW6-GND-Pad0)
- SW7 pad 0: (no net) -> unconnected-(SW7-GND-Pad0)
- SW8 pad 0: (no net) -> unconnected-(SW8-GND-Pad0)
- SW9 pad 0: (no net) -> unconnected-(SW9-GND-Pad0)
Other:
- outline, holes or cut-outs redrawn
