File: pcb/c51keypad/c51keypad.kicad_sch (KiCad schematic)
At the start: 49 parts, among them CN1 PZ254V-11-04P, J1 USB_C_Receptacle_USB2.0_16P, U1 CH9328, U2 STC12C5604AD-35I-DIP20, Y1 Crystal_12MHZ

Commit message: stc15
Parts:
- removed C3: 10uF, Capacitor_SMD:C_0603_1608Metric_Pad1.08x0.95mm_HandSolder, symbol Device:C
- removed C6, C7: 20pF, Capacitor_SMD:C_0603_1608Metric_Pad1.08x0.95mm_HandSolder, symbol Device:C
- removed R3: 1k, Resistor_SMD:R_0603_1608Metric_Pad0.98x0.95mm_HandSolder, symbol Device:R
- removed U2: STC12C5604AD-35I-DIP20, Package_DIP:DIP-20_W7.62mm_Socket_LongPads, symbol Custom_Library:STC12C5604AD-35I-DIP20
- removed Y1: Crystal_12MHZ, Crystal:Crystal_SMD_3225-4Pin_3.2x2.5mm_HandSoldering, symbol Device:Crystal_GND24
- added U2: STC15W204S-35I-SOP16, Package_SO:SOP-16_3.9x9.9mm_P1.27mm, symbol Custom_Library:STC15W204S-35I-SOP16
Connections:
- net COL0: now also U2.11 (P3.2/INT0)
- net COL1: now also U2.12 (P3.3/INT1)
- net COL2: now also U2.13 (P3.6/INT2#/RXD_2)
- net COL3: now also U2.14 (P3.7/INT3#/TXD_2)
- net GND: now also J1.13 (GND), U1.11 (IO2), U2.8 (GND); no longer U1.14 (IO3)
- net ROW0: now also U2.15 (P1.0/RSTOUT_LOW)
- net ROW1: now also U2.16 (P1.1)
- net ROW2: now also U2.1 (CMPO/T0/P1.2)
- net ROW3: now also U2.2 (P1.3)
- net ROW4: now also U2.3 (T0CLKO/P1.4)
- net RXD: now also U2.9 (P3.0/RxD/INT4#/T2CLKO)
- net TXD: now also U2.10 (P3.1/TxD/T2)
- net VBUS: now also U1.14 (IO3), U2.6 (VCC); no longer U1.11 (IO2)
- no-connect marks 10 -> 9
Other:
- moved on the sheet: C4, C5, CN1

Commit message: 内存优化
Connections:
- net RXD: no longer U1.2 (TXD)
- no-connect marks 9 -> 10
Changed lines of the file:
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@@
+	)
+	(no_connect
+		(at 119.38 38.1)
 	)
 	(no_connect
@@
 		(pts
 			(xy 193.04 52.07) (xy 193.04 55.88)
-		)
-		(stroke
-			(width 0)
-			(type default)
-		)
-	)
-	(wire
-		(pts
-			(xy 113.03 38.1) (xy 119.38 38.1)
 		)
 		(stroke
@@
 		(fields_autoplaced yes)
 		(effects
-			(font
-				(size 1.27 1.27)
-			)
-			(justify left bottom)
-		)
-	)
-	(label "RXD"
-		(at 113.03 38.1 0)
-		(fields_autoplaced yes)
-		(effects
